File: Roto-Pad-2.0/logicshifter.kicad_sch (KiCad schematic)
At the start: 3 parts, among them Q1 BSS138

Commit message: layout completed, first draft of routing
Parts:
- R11, R8: footprint (none) -> PCM_4ms_Resistor:R_0402
Changed lines of the file:
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@@
 			)
 		)
-		(property "Footprint" ""
+		(property "Footprint" "PCM_4ms_Resistor:R_0402"
 			(at 63.5 68.58 0)
 			(effects
@@
 			)
 		)
-		(property "Footprint" ""
+		(property "Footprint" "PCM_4ms_Resistor:R_0402"
 			(at 96.52 68.58 0)
 			(effects
