File: Roto-Pad-2.0/Roto-Pad-2.0.kicad_pcb (KiCad board)
At the start: 2 copper layers, 3.8 x 3.4 mm, 89 parts, among them SW1 Switch, SW10 Switch, SW11 Switch, SW12 Switch, SW13 Switch, SW14 Switch, SW15 Switch, SW16 Switch, SW17 Switch, SW18 Switch, SW19 Switch, SW2 Switch, SW20 Switch, SW21 Switch, SW22 Switch, SW23 Switch, SW24 Switch, SW25 Switch, SW3 Switch, SW4 Switch, SW5 Switch, SW6 Switch, SW7 Switch, SW8 Switch, SW9 Switch, U1 Pico

Commit message: completed physical PCB layout
Parts:
- removed the D25 at (217.9, 73.8)
- removed the LED25 at (289.1, 63.8)
- removed LED26, LED27, LED28, LED29, LED30: SK6812, Custom:SK6812-Mini-E MX
- added D1: D, PCM_Diode_SMD_AKL:D_1206_3216Metric_Castellated, B.Cu at (50.2, 65.0)
- added LED1: SK6812, Custom:SK6812-Mini-E MX, F.Cu at (58.4, 62.4)
- R1, R2, R3, R4, R5, R6, R7: moved to B.Cu
- moved LED21 210.5 mm to (58.4, 138.4)
- moved LED16 207.1 mm to (58.4, 119.4)
- moved LED11 204.1 mm to (58.4, 100.4)
- moved LED6 201.6 mm to (58.4, 81.4)
- moved LED22 200.6 mm to (77.4, 138.4)
- moved LED17 197.1 mm to (77.4, 119.4)
- moved LED12 194.0 mm to (77.4, 100.4)
- moved LED7 191.4 mm to (77.4, 81.4)
- moved LED23 190.9 mm to (96.4, 138.4)
- moved LED2 189.3 mm to (77.4, 62.4)
- moved LED18 187.1 mm to (96.4, 119.4)
- moved D6 186.1 mm to (50.2, 84.0)
- moved LED13 183.8 mm to (96.4, 100.4)
- moved D16 182.7 mm to (50.2, 122.0)
- moved D11 182.3 mm to (50.2, 103.0)
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- renumbered D1 to D25, LED1 to LED25
Connections:
- D10 pad 1: /Key Matrix/Col 5 -> /Key Matrix/Col 1
- D10 pad 2: Net-(D10-A+) -> Net-(D1-A+)
- D11 pad 2: Net-(D11-A+) -> Net-(D1-A+)
- D12 pad 1: /Key Matrix/Col 2 -> /Key Matrix/Col 1
- D12 pad 2: Net-(D12-A+) -> Net-(D1-A+)
- D13 pad 1: /Key Matrix/Col 4 -> /Key Matrix/Col 1
- D13 pad 2: Net-(D13-A+) -> Net-(D1-A+)
- D14 pad 1: /Key Matrix/Col 3 -> /Key Matrix/Col 1
- D14 pad 2: Net-(D14-A+) -> Net-(D1-A+)
- D15 pad 1: /Key Matrix/Col 5 -> /Key Matrix/Col 1
- D15 pad 2: Net-(D15-A+) -> Net-(D1-A+)
- D16 pad 2: Net-(D16-A+) -> Net-(D1-A+)
- D17 pad 1: /Key Matrix/Col 2 -> /Key Matrix/Col 1
- D17 pad 2: Net-(D17-A+) -> Net-(D1-A+)
- D18 pad 1: /Key Matrix/Col 4 -> /Key Matrix/Col 1
- D18 pad 2: Net-(D18-A+) -> Net-(D1-A+)
- D19 pad 1: /Key Matrix/Col 3 -> /Key Matrix/Col 1
- D19 pad 2: Net-(D19-A+) -> Net-(D1-A+)
- D2 pad 1: /Key Matrix/Col 2 -> /Key Matrix/Col 1
- D2 pad 2: Net-(D2-A+) -> Net-(D1-A+)
- D20 pad 1: /Key Matrix/Col 5 -> /Key Matrix/Col 1
- D20 pad 2: Net-(D20-A+) -> Net-(D1-A+)
- D21 pad 2: Net-(D21-A+) -> Net-(D1-A+)
- D22 pad 1: /Key Matrix/Col 2 -> /Key Matrix/Col 1
- D22 pad 2: Net-(D22-A+) -> Net-(D1-A+)
- D23 pad 1: /Key Matrix/Col 4 -> /Key Matrix/Col 1
- D23 pad 2: Net-(D23-A+) -> Net-(D1-A+)
- D24 pad 1: /Key Matrix/Col 3 -> /Key Matrix/Col 1
- D24 pad 2: Net-(D24-A+) -> Net-(D1-A+)
- D3 pad 1: /Key Matrix/Col 4 -> /Key Matrix/Col 1
- D3 pad 2: Net-(D3-A+) -> Net-(D1-A+)
- D4 pad 1: /Key Matrix/Col 3 -> /Key Matrix/Col 1
- D4 pad 2: Net-(D4-A+) -> Net-(D1-A+)
- D5 pad 1: /Key Matrix/Col 5 -> /Key Matrix/Col 1
- D5 pad 2: Net-(D5-A+) -> Net-(D1-A+)
- D6 pad 2: Net-(D6-A+) -> Net-(D1-A+)
- D7 pad 1: /Key Matrix/Col 2 -> /Key Matrix/Col 1
- D7 pad 2: Net-(D7-A+) -> Net-(D1-A+)
- D8 pad 1: /Key Matrix/Col 4 -> /Key Matrix/Col 1
- D8 pad 2: Net-(D8-A+) -> Net-(D1-A+)
- D9 pad 1: /Key Matrix/Col 3 -> /Key Matrix/Col 1
- D9 pad 2: Net-(D9-A+) -> Net-(D1-A+)
- LED10 pad 2: Net-(LED10-DOUT) -> Net-(LED1-DOUT)
- LED10 pad 4: Net-(LED10-DIN) -> /Neopixel/DIN
- LED11 pad 2: Net-(LED11-DOUT) -> Net-(LED1-DOUT)
- LED11 pad 4: Net-(LED10-DOUT) -> /Neopixel/DIN
- LED12 pad 2: Net-(LED12-DOUT) -> Net-(LED1-DOUT)
- LED12 pad 4: Net-(LED11-DOUT) -> /Neopixel/DIN
- LED13 pad 2: Net-(LED13-DOUT) -> Net-(LED1-DOUT)
- LED13 pad 4: Net-(LED12-DOUT) -> /Neopixel/DIN
- LED14 pad 2: Net-(LED14-DOUT) -> Net-(LED1-DOUT)
- LED14 pad 4: Net-(LED13-DOUT) -> /Neopixel/DIN
- LED15 pad 2: Net-(LED15-DOUT) -> Net-(LED1-DOUT)
- LED15 pad 4: Net-(LED14-DOUT) -> /Neopixel/DIN
- LED16 pad 2: Net-(LED16-DOUT) -> Net-(LED1-DOUT)
- LED16 pad 4: Net-(LED15-DOUT) -> /Neopixel/DIN
- LED17 pad 2: Net-(LED17-DOUT) -> Net-(LED1-DOUT)
- LED17 pad 4: Net-(LED16-DOUT) -> /Neopixel/DIN
- LED18 pad 2: Net-(LED18-DOUT) -> Net-(LED1-DOUT)
- LED18 pad 4: Net-(LED17-DOUT) -> /Neopixel/DIN
- LED19 pad 2: Net-(LED19-DOUT) -> Net-(LED1-DOUT)
- LED19 pad 4: Net-(LED18-DOUT) -> /Neopixel/DIN
- LED2 pad 2: Net-(LED2-DOUT) -> Net-(LED1-DOUT)
- LED2 pad 4: Net-(LED1-DOUT) -> /Neopixel/DIN
- LED20 pad 2: Net-(LED20-DOUT) -> Net-(LED1-DOUT)
- LED20 pad 4: Net-(LED19-DOUT) -> /Neopixel/DIN
- LED21 pad 2: Net-(LED21-DOUT) -> Net-(LED1-DOUT)
- LED21 pad 4: Net-(LED20-DOUT) -> /Neopixel/DIN
- LED22 pad 2: Net-(LED22-DOUT) -> Net-(LED1-DOUT)
- LED22 pad 4: Net-(LED21-DOUT) -> /Neopixel/DIN
- LED23 pad 2: Net-(LED23-DOUT) -> Net-(LED1-DOUT)
- LED23 pad 4: Net-(LED22-DOUT) -> /Neopixel/DIN
- LED24 pad 2: Net-(LED24-DOUT) -> Net-(LED1-DOUT)
- LED24 pad 4: Net-(LED23-DOUT) -> /Neopixel/DIN
- LED3 pad 2: Net-(LED3-DOUT) -> Net-(LED1-DOUT)
- LED3 pad 4: Net-(LED2-DOUT) -> /Neopixel/DIN
- LED4 pad 2: Net-(LED4-DOUT) -> Net-(LED1-DOUT)
- LED4 pad 4: Net-(LED3-DOUT) -> /Neopixel/DIN
- LED5 pad 2: Net-(LED5-DOUT) -> Net-(LED1-DOUT)
- LED5 pad 4: Net-(LED4-DOUT) -> /Neopixel/DIN
- LED6 pad 2: Net-(LED6-DOUT) -> Net-(LED1-DOUT)
- LED6 pad 4: Net-(LED5-DOUT) -> /Neopixel/DIN
- LED7 pad 2: Net-(LED7-DOUT) -> Net-(LED1-DOUT)
- LED7 pad 4: Net-(LED6-DOUT) -> /Neopixel/DIN
- LED8 pad 2: Net-(LED8-DOUT) -> Net-(LED1-DOUT)
- LED8 pad 4: Net-(LED7-DOUT) -> /Neopixel/DIN
- LED9 pad 2: Net-(LED10-DIN) -> Net-(LED1-DOUT)
- LED9 pad 4: Net-(LED8-DOUT) -> /Neopixel/DIN

Commit message: added more heirarchical sheets, debouncing
Parts:
- removed E2: ENCODER-RGB-SWITCH, Custom:Led Encoder
- added C1: C104, Keebio-Parts.pretty-master:C_0402, F.Cu at (-63.0, 109.0)
- added C2: C104, Keebio-Parts.pretty-master:C_0402, F.Cu at (-70.5, 109.0)
- added LED26: SK6812, Custom:SK6812-Mini-E MX, F.Cu at (-124.5, 108.4)
- added LED27: SK6812, Custom:SK6812-Mini-E MX, F.Cu at (-116.1, 108.4)
- added LED28: SK6812, Custom:SK6812-Mini-E MX, F.Cu at (-107.6, 108.4)
- added LED29: SK6812, Custom:SK6812-Mini-E MX, F.Cu at (-99.2, 108.4)
- added LED30: SK6812, Custom:SK6812-Mini-E MX, F.Cu at (-90.7, 108.4)
- added S1: ENCODER-RGB-SWITCH, Custom:Led Encoder, F.Cu at (134.5, 39.0)
- D1, D10, D11, D12, D13, D14, D15, D16, D17, D18, D19, D2, D20, D21, D22, D23, D24, D25, D3, D4, D5, D6, D7, D8, D9: footprint PCM_Diode_SMD_AKL:D_1206_3216Metric_Castellated -> Keebio-Parts.pretty-master:Diode-dual
- moved D10 13.7 mm to (135.0, 73.5)
- moved D12 13.7 mm to (78.0, 92.5)
- moved D13 13.7 mm to (97.0, 92.5)
- moved D14 13.7 mm to (116.0, 92.5)
- moved D15 13.7 mm to (135.0, 92.5)
- moved D17 13.7 mm to (78.0, 111.5)
- moved D18 13.7 mm to (97.0, 111.5)
- moved D19 13.7 mm to (116.0, 111.5)
- moved D2 13.7 mm to (78.0, 54.5)
- moved D20 13.7 mm to (135.0, 111.5)
- moved D22 13.7 mm to (78.0, 130.5)
- moved D23 13.7 mm to (97.0, 130.5)
- moved D24 13.7 mm to (116.0, 130.5)
- moved D25 13.7 mm to (135.0, 130.5)
- moved D3 13.7 mm to (97.0, 54.5)
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Connections:
- D10 pad 1: /Key Matrix/Col 1 -> /Key Matrix/Col 5
- D10 pad 2: Net-(D1-A+) -> Net-(D10-A+)
- D11 pad 2: Net-(D1-A+) -> Net-(D11-A+)
- D12 pad 1: /Key Matrix/Col 1 -> /Key Matrix/Col 2
- D12 pad 2: Net-(D1-A+) -> Net-(D12-A+)
- D13 pad 1: /Key Matrix/Col 1 -> /Key Matrix/Col 4
- D13 pad 2: Net-(D1-A+) -> Net-(D13-A+)
- D14 pad 1: /Key Matrix/Col 1 -> /Key Matrix/Col 3
- D14 pad 2: Net-(D1-A+) -> Net-(D14-A+)
- D15 pad 1: /Key Matrix/Col 1 -> /Key Matrix/Col 5
- D15 pad 2: Net-(D1-A+) -> Net-(D15-A+)
- D16 pad 2: Net-(D1-A+) -> Net-(D16-A+)
- D17 pad 1: /Key Matrix/Col 1 -> /Key Matrix/Col 2
- D17 pad 2: Net-(D1-A+) -> Net-(D17-A+)
- D18 pad 1: /Key Matrix/Col 1 -> /Key Matrix/Col 4
- D18 pad 2: Net-(D1-A+) -> Net-(D18-A+)
- D19 pad 1: /Key Matrix/Col 1 -> /Key Matrix/Col 3
- D19 pad 2: Net-(D1-A+) -> Net-(D19-A+)
- D2 pad 1: /Key Matrix/Col 1 -> /Key Matrix/Col 2
- D2 pad 2: Net-(D1-A+) -> Net-(D2-A+)
- D20 pad 1: /Key Matrix/Col 1 -> /Key Matrix/Col 5
- D20 pad 2: Net-(D1-A+) -> Net-(D20-A+)
- D21 pad 2: Net-(D1-A+) -> Net-(D21-A+)
- D22 pad 1: /Key Matrix/Col 1 -> /Key Matrix/Col 2
- D22 pad 2: Net-(D1-A+) -> Net-(D22-A+)
- D23 pad 1: /Key Matrix/Col 1 -> /Key Matrix/Col 4
- D23 pad 2: Net-(D1-A+) -> Net-(D23-A+)
- D24 pad 1: /Key Matrix/Col 1 -> /Key Matrix/Col 3
- D24 pad 2: Net-(D1-A+) -> Net-(D24-A+)
- D25 pad 1: /Key Matrix/Col 1 -> /Key Matrix/Col 5
- D25 pad 2: Net-(D1-A+) -> Net-(D25-A+)
- D3 pad 1: /Key Matrix/Col 1 -> /Key Matrix/Col 4
- D3 pad 2: Net-(D1-A+) -> Net-(D3-A+)
- D4 pad 1: /Key Matrix/Col 1 -> /Key Matrix/Col 3
- D4 pad 2: Net-(D1-A+) -> Net-(D4-A+)
- D5 pad 1: /Key Matrix/Col 1 -> /Key Matrix/Col 5
- D5 pad 2: Net-(D1-A+) -> Net-(D5-A+)
- D6 pad 2: Net-(D1-A+) -> Net-(D6-A+)
- D7 pad 1: /Key Matrix/Col 1 -> /Key Matrix/Col 2
- D7 pad 2: Net-(D1-A+) -> Net-(D7-A+)
- D8 pad 1: /Key Matrix/Col 1 -> /Key Matrix/Col 4
- D8 pad 2: Net-(D1-A+) -> Net-(D8-A+)
- D9 pad 1: /Key Matrix/Col 1 -> /Key Matrix/Col 3
- D9 pad 2: Net-(D1-A+) -> Net-(D9-A+)
- LED10 pad 2: Net-(LED1-DOUT) -> Net-(LED10-DOUT)
- LED10 pad 4: /Neopixel/DIN -> Net-(LED10-DIN)
- LED11 pad 2: Net-(LED1-DOUT) -> Net-(LED11-DOUT)
- LED11 pad 4: /Neopixel/DIN -> Net-(LED10-DOUT)
- LED12 pad 2: Net-(LED1-DOUT) -> Net-(LED12-DOUT)
- LED12 pad 4: /Neopixel/DIN -> Net-(LED11-DOUT)
- LED13 pad 2: Net-(LED1-DOUT) -> Net-(LED13-DOUT)
- LED13 pad 4: /Neopixel/DIN -> Net-(LED12-DOUT)
- LED14 pad 2: Net-(LED1-DOUT) -> Net-(LED14-DOUT)
- LED14 pad 4: /Neopixel/DIN -> Net-(LED13-DOUT)
- LED15 pad 2: Net-(LED1-DOUT) -> Net-(LED15-DOUT)
- LED15 pad 4: /Neopixel/DIN -> Net-(LED14-DOUT)
- LED16 pad 2: Net-(LED1-DOUT) -> Net-(LED16-DOUT)
- LED16 pad 4: /Neopixel/DIN -> Net-(LED15-DOUT)
- LED17 pad 2: Net-(LED1-DOUT) -> Net-(LED17-DOUT)
- LED17 pad 4: /Neopixel/DIN -> Net-(LED16-DOUT)
- LED18 pad 2: Net-(LED1-DOUT) -> Net-(LED18-DOUT)
- LED18 pad 4: /Neopixel/DIN -> Net-(LED17-DOUT)
- LED19 pad 2: Net-(LED1-DOUT) -> Net-(LED19-DOUT)
- LED19 pad 4: /Neopixel/DIN -> Net-(LED18-DOUT)
- LED2 pad 2: Net-(LED1-DOUT) -> Net-(LED2-DOUT)
- LED2 pad 4: /Neopixel/DIN -> Net-(LED1-DOUT)
- LED20 pad 2: Net-(LED1-DOUT) -> Net-(LED20-DOUT)
- LED20 pad 4: /Neopixel/DIN -> Net-(LED19-DOUT)
- LED21 pad 2: Net-(LED1-DOUT) -> Net-(LED21-DOUT)
- LED21 pad 4: /Neopixel/DIN -> Net-(LED20-DOUT)
- LED22 pad 2: Net-(LED1-DOUT) -> Net-(LED22-DOUT)
- LED22 pad 4: /Neopixel/DIN -> Net-(LED21-DOUT)
- LED23 pad 2: Net-(LED1-DOUT) -> Net-(LED23-DOUT)
- LED23 pad 4: /Neopixel/DIN -> Net-(LED22-DOUT)
- LED24 pad 2: Net-(LED1-DOUT) -> Net-(LED24-DOUT)
- LED24 pad 4: /Neopixel/DIN -> Net-(LED23-DOUT)
- LED25 pad 2: Net-(LED1-DOUT) -> Net-(LED25-DOUT)
- LED25 pad 4: /Neopixel/DIN -> Net-(LED24-DOUT)
- LED3 pad 2: Net-(LED1-DOUT) -> Net-(LED3-DOUT)
- LED3 pad 4: /Neopixel/DIN -> Net-(LED2-DOUT)
- LED4 pad 2: Net-(LED1-DOUT) -> Net-(LED4-DOUT)
- LED4 pad 4: /Neopixel/DIN -> Net-(LED3-DOUT)
- LED5 pad 2: Net-(LED1-DOUT) -> Net-(LED5-DOUT)
- LED5 pad 4: /Neopixel/DIN -> Net-(LED4-DOUT)
- LED6 pad 2: Net-(LED1-DOUT) -> Net-(LED6-DOUT)
- LED6 pad 4: /Neopixel/DIN -> Net-(LED5-DOUT)
- LED7 pad 2: Net-(LED1-DOUT) -> Net-(LED7-DOUT)
- LED7 pad 4: /Neopixel/DIN -> Net-(LED6-DOUT)
- LED8 pad 2: Net-(LED1-DOUT) -> Net-(LED8-DOUT)
- LED8 pad 4: /Neopixel/DIN -> Net-(LED7-DOUT)
- LED9 pad 2: Net-(LED1-DOUT) -> Net-(LED10-DIN)
- LED9 pad 4: /Neopixel/DIN -> Net-(LED8-DOUT)
- SW10 pad 1: /Key Matrix/Row 1 -> /Key Matrix/Row 2
- SW10 pad 2: Net-(D1-A+) -> Net-(D10-A+)
- SW11 pad 1: /Key Matrix/Row 1 -> /Key Matrix/Row 3
- SW11 pad 2: Net-(D1-A+) -> Net-(D11-A+)
- SW12 pad 1: /Key Matrix/Row 1 -> /Key Matrix/Row 3
- SW12 pad 2: Net-(D1-A+) -> Net-(D12-A+)
- SW13 pad 1: /Key Matrix/Row 1 -> /Key Matrix/Row 3
- SW13 pad 2: Net-(D1-A+) -> Net-(D13-A+)
- SW14 pad 1: /Key Matrix/Row 1 -> /Key Matrix/Row 3
- SW14 pad 2: Net-(D1-A+) -> Net-(D14-A+)
- SW15 pad 1: /Key Matrix/Row 1 -> /Key Matrix/Row 3
- SW15 pad 2: Net-(D1-A+) -> Net-(D15-A+)
- SW16 pad 1: /Key Matrix/Row 1 -> /Key Matrix/Row 4
- SW16 pad 2: Net-(D1-A+) -> Net-(D16-A+)
- SW17 pad 1: /Key Matrix/Row 1 -> /Key Matrix/Row 4
- SW17 pad 2: Net-(D1-A+) -> Net-(D17-A+)
- SW18 pad 1: /Key Matrix/Row 1 -> /Key Matrix/Row 4
- SW18 pad 2: Net-(D1-A+) -> Net-(D18-A+)
- SW19 pad 1: /Key Matrix/Row 1 -> /Key Matrix/Row 4
- SW19 pad 2: Net-(D1-A+) -> Net-(D19-A+)
- SW2 pad 2: Net-(D1-A+) -> Net-(D2-A+)
- SW20 pad 1: /Key Matrix/Row 1 -> /Key Matrix/Row 4
- SW20 pad 2: Net-(D1-A+) -> Net-(D20-A+)
- SW21 pad 1: /Key Matrix/Row 1 -> /Key Matrix/Row 5
- SW21 pad 2: Net-(D1-A+) -> Net-(D21-A+)
- SW22 pad 1: /Key Matrix/Row 1 -> /Key Matrix/Row 5
- SW22 pad 2: Net-(D1-A+) -> Net-(D22-A+)
- SW23 pad 1: /Key Matrix/Row 1 -> /Key Matrix/Row 5
- SW23 pad 2: Net-(D1-A+) -> Net-(D23-A+)
- SW24 pad 1: /Key Matrix/Row 1 -> /Key Matrix/Row 5
- SW24 pad 2: Net-(D1-A+) -> Net-(D24-A+)
- SW25 pad 1: /Key Matrix/Row 1 -> /Key Matrix/Row 5
- SW25 pad 2: Net-(D1-A+) -> Net-(D25-A+)
- SW3 pad 2: Net-(D1-A+) -> Net-(D3-A+)
- SW4 pad 2: Net-(D1-A+) -> Net-(D4-A+)
- SW5 pad 2: Net-(D1-A+) -> Net-(D5-A+)
- SW6 pad 1: /Key Matrix/Row 1 -> /Key Matrix/Row 2
- SW6 pad 2: Net-(D1-A+) -> Net-(D6-A+)
- SW7 pad 1: /Key Matrix/Row 1 -> /Key Matrix/Row 2
- SW7 pad 2: Net-(D1-A+) -> Net-(D7-A+)
- SW8 pad 1: /Key Matrix/Row 1 -> /Key Matrix/Row 2
- SW8 pad 2: Net-(D1-A+) -> Net-(D8-A+)
- SW9 pad 1: /Key Matrix/Row 1 -> /Key Matrix/Row 2
- SW9 pad 2: Net-(D1-A+) -> Net-(D9-A+)
- U1 pad 38: /Neopixel/GND -> unconnected-(U1-GND-Pad38)
Routing:
- net Net-(LED20-DOUT): track 0.00 -> 104.1 mm
- net Net-(LED5-DOUT): track 0.00 -> 103.8 mm
- net Net-(LED15-DOUT): track 0.00 -> 103.6 mm
- net Net-(LED10-DOUT): track 0.00 -> 103.6 mm
- net /Key Matrix/Col 1: track 0.00 -> 86.4 mm
- net /Key Matrix/Col 4: track 0.00 -> 85.6 mm
- net /Key Matrix/Col 3: track 0.00 -> 85.6 mm
- net /Key Matrix/Col 2: track 0.00 -> 85.6 mm
- net /Key Matrix/Row 2: track 0.00 -> 82.4 mm
- net /Key Matrix/Row 5: track 0.00 -> 82.3 mm
- net /Key Matrix/Row 1: track 0.00 -> 82.3 mm
- net /Key Matrix/Row 4: track 0.00 -> 82.3 mm
- net /Key Matrix/Row 3: track 0.00 -> 82.2 mm
- net /Key Matrix/Col 5: track 0.00 -> 64.2 mm
- net Net-(LED10-DIN): track 0.00 -> 29.4 mm
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
Commit message: layout completed, first draft of routing
Parts:
- removed C2: C104, Keebio-Parts.pretty-master:C_0402
- removed R1, R2, R3: 220ohm, PCM_Resistor_SMD_AKL:R_1206_3216Metric
- removed R4, R5, R6, R7: R 10k, PCM_Resistor_SMD_AKL:R_1206_3216Metric
- removed S1: ENCODER-RGB-SWITCH, Custom:Led Encoder
- added C10: 10nf, Keebio-Parts.pretty-master:C_0402, F.Cu at (125.0, 47.5)
- added C11: 10nf, Keebio-Parts.pretty-master:C_0402, F.Cu at (125.0, 39.0)
- added C12: 100nf, Keebio-Parts.pretty-master:C_0402, F.Cu at (119.0, 36.5)
- added C5: 100nf, Keebio-Parts.pretty-master:C_0402, B.Cu at (106.0, 42.0)
- added C6: 100nf, Keebio-Parts.pretty-master:C_0402, B.Cu at (110.0, 42.0)
- added C7: 100nf, Keebio-Parts.pretty-master:C_0402, B.Cu at (117.0, 42.0)
- added C8: 100nf, Keebio-Parts.pretty-master:C_0402, B.Cu at (113.5, 42.0)
- added C9: 100nf, Keebio-Parts.pretty-master:C_0402, B.Cu at (120.5, 42.0)
- added LED31: SK6812, PCM_LED_SMD_AKL:LED_SK6812_EC15_1.5x1.5mm, B.Cu at (78.0, 25.5)
- added LED32: SK6812, PCM_LED_SMD_AKL:LED_SK6812_EC15_1.5x1.5mm, B.Cu at (119.0, 25.5)
- added LED33: SK6812, PCM_LED_SMD_AKL:LED_SK6812_EC15_1.5x1.5mm, B.Cu at (145.5, 51.5)
- added LED34: SK6812, PCM_LED_SMD_AKL:LED_SK6812_EC15_1.5x1.5mm, B.Cu at (145.5, 93.5)
- added LED35: SK6812, PCM_LED_SMD_AKL:LED_SK6812_EC15_1.5x1.5mm, B.Cu at (145.5, 131.5)
- added Q1: BSS138, PCM_Package_TO_SOT_SMD_AKL:SOT-23, B.Cu at (58.5, 38.5)
- added R10: 500, adafruit:R1206, B.Cu at (53.0, 52.0)
- added R11: 10k, PCM_4ms_Resistor:R_0402, B.Cu at (63.0, 39.5)
- added R14: 50, adafruit:R0805, B.Cu at (106.0, 47.5)
- added R15: 50, adafruit:R0805, B.Cu at (110.0, 47.5)
- added R16: 50, adafruit:R0805, B.Cu at (117.0, 47.5)
- added R17: 50, adafruit:R0805, B.Cu at (113.5, 47.5)
- added R18: 50, adafruit:R0805, B.Cu at (120.5, 47.5)
- added R19: R 10k, PCM_4ms_Resistor:R_0402, F.Cu at (125.0, 46.0)
- added R20: R 10k, PCM_4ms_Resistor:R_0402, F.Cu at (125.0, 40.5)
- added R21: R 10k, PCM_4ms_Resistor:R_0402, F.Cu at (125.0, 44.5)
- added R22: R 10k, PCM_4ms_Resistor:R_0402, F.Cu at (125.0, 42.0)
- added R23: 50, adafruit:R0805, F.Cu at (124.0, 35.5)
- added R24: 220ohm, adafruit:R1206, F.Cu at (123.5, 33.0)
- added R25: 220ohm, adafruit:R1206, F.Cu at (123.5, 28.0)
- added R26: 220ohm, adafruit:R1206, F.Cu at (123.5, 30.5)
- added R27: 2.2k, PCM_4ms_Resistor:R_0402, F.Cu at (119.0, 35.0)
- added R8: 10k, PCM_4ms_Resistor:R_0402, B.Cu at (63.0, 37.0)
- added R9: 500, adafruit:R1206, B.Cu at (140.5, 126.0)
- added S2: ENCODER-RGB-SWITCH, Custom:Led Encoder, F.Cu at (135.5, 37.0)
- C1: value C104 -> C-polar 1000uf; footprint Keebio-Parts.pretty-master:C_0402 -> Capacitors:NIC_10X10.5_CAP
- D1, D10, D11, D12, D13, D14, D15, D16, D17, D18, D19, D2, D20, D21, D22, D23, D24, D25, D3, D4, D5, D6, D7, D8, D9: footprint Keebio-Parts.pretty-master:Diode-dual -> PCM_Diode_SMD_AKL:D_SMA
- LED26, LED27, LED28, LED29, LED30: footprint Custom:SK6812-Mini-E MX -> PCM_LED_SMD_AKL:LED_SK6812_EC15_1.5x1.5mm; moved to B.Cu
- moved LED26 245.7 mm to (118.0, 148.0), turned to 90 degrees
- moved LED27 200.0 mm to (80.0, 148.0), turned to 90 degrees
- moved C1 187.9 mm to (109.5, 34.5), turned to 180 degrees
- moved LED28 157.9 mm to (48.5, 132.0), turned to -90 degrees
- moved LED30 149.8 mm to (48.5, 53.0), turned to -90 degrees
- moved LED29 148.3 mm to (48.5, 95.0), turned to -90 degrees
- moved D1 15.3 mm to (54.0, 69.0), turned to 0 degrees
- moved D10 15.3 mm to (130.0, 88.0), turned to 0 degrees
- moved D11 15.3 mm to (54.0, 107.0), turned to 0 degrees
- moved D12 15.3 mm to (73.0, 107.0), turned to 0 degrees
- moved D13 15.3 mm to (92.0, 107.0), turned to 0 degrees
- moved D14 15.3 mm to (111.0, 107.0), turned to 0 degrees
- moved D15 15.3 mm to (130.0, 107.0), turned to 0 degrees
- moved D16 15.3 mm to (54.0, 126.0), turned to 0 degrees
- moved D17 15.3 mm to (73.0, 126.0), turned to 0 degrees
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Connections:
- net /Neopixel/5v renamed 5v
- D1 pad 1: /Key Matrix/Col 1 -> /Debounce Array/input 1
- D10 pad 1: /Key Matrix/Col 5 -> /Debounce Array/input 5
- D11 pad 1: /Key Matrix/Col 1 -> /Debounce Array/input 1
- D12 pad 1: /Key Matrix/Col 2 -> /Debounce Array/input 2
- D13 pad 1: /Key Matrix/Col 4 -> /Debounce Array/input 4
- D14 pad 1: /Key Matrix/Col 3 -> /Debounce Array/input 3
- D15 pad 1: /Key Matrix/Col 5 -> /Debounce Array/input 5
- D16 pad 1: /Key Matrix/Col 1 -> /Debounce Array/input 1
- D17 pad 1: /Key Matrix/Col 2 -> /Debounce Array/input 2
- D18 pad 1: /Key Matrix/Col 4 -> /Debounce Array/input 4
- D19 pad 1: /Key Matrix/Col 3 -> /Debounce Array/input 3
- D2 pad 1: /Key Matrix/Col 2 -> /Debounce Array/input 2
- D20 pad 1: /Key Matrix/Col 5 -> /Debounce Array/input 5
- D21 pad 1: /Key Matrix/Col 1 -> /Debounce Array/input 1
- D22 pad 1: /Key Matrix/Col 2 -> /Debounce Array/input 2
- D23 pad 1: /Key Matrix/Col 4 -> /Debounce Array/input 4
- D24 pad 1: /Key Matrix/Col 3 -> /Debounce Array/input 3
- D25 pad 1: /Key Matrix/Col 5 -> /Debounce Array/input 5
- D3 pad 1: /Key Matrix/Col 4 -> /Debounce Array/input 4
- D4 pad 1: /Key Matrix/Col 3 -> /Debounce Array/input 3
- D5 pad 1: /Key Matrix/Col 5 -> /Debounce Array/input 5
- D6 pad 1: /Key Matrix/Col 1 -> /Debounce Array/input 1
- D7 pad 1: /Key Matrix/Col 2 -> /Debounce Array/input 2
- D8 pad 1: /Key Matrix/Col 4 -> /Debounce Array/input 4
- D9 pad 1: /Key Matrix/Col 3 -> /Debounce Array/input 3
- LED1 pad 3: /Neopixel/GND -> GND
- LED1 pad 4: /Neopixel/DIN -> Net-(LED1-DIN)
- LED10 pad 3: /Neopixel/GND -> GND
- LED11 pad 3: /Neopixel/GND -> GND
- LED12 pad 3: /Neopixel/GND -> GND
- LED13 pad 3: /Neopixel/GND -> GND
- LED14 pad 3: /Neopixel/GND -> GND
- LED15 pad 3: /Neopixel/GND -> GND
- LED16 pad 3: /Neopixel/GND -> GND
- LED17 pad 3: /Neopixel/GND -> GND
- LED18 pad 3: /Neopixel/GND -> GND
- LED19 pad 3: /Neopixel/GND -> GND
- LED2 pad 3: /Neopixel/GND -> GND
- LED20 pad 3: /Neopixel/GND -> GND
- LED21 pad 3: /Neopixel/GND -> GND
- LED22 pad 3: /Neopixel/GND -> GND
- LED23 pad 3: /Neopixel/GND -> GND
- LED24 pad 3: /Neopixel/GND -> GND
- LED25 pad 3: /Neopixel/GND -> GND
- LED26 pad 3: /Neopixel/GND -> GND
- LED27 pad 3: /Neopixel/GND -> GND
- LED28 pad 3: /Neopixel/GND -> GND
- LED29 pad 3: /Neopixel/GND -> GND
- LED3 pad 3: /Neopixel/GND -> GND
- LED30 pad 2: unconnected-(LED30-DOUT-Pad2) -> Net-(LED30-DOUT)
- LED30 pad 3: /Neopixel/GND -> GND
- LED4 pad 3: /Neopixel/GND -> GND
- LED5 pad 3: /Neopixel/GND -> GND
- LED6 pad 3: /Neopixel/GND -> GND
- LED7 pad 3: /Neopixel/GND -> GND
- LED8 pad 3: /Neopixel/GND -> GND
- LED9 pad 3: /Neopixel/GND -> GND
- U1 pad 10: /Key Matrix/Col 3 -> /Debounce Array/output 3
- U1 pad 13: /Neopixel/GND -> GND
- U1 pad 17: /Key Matrix/Col 4 -> /Debounce Array/output 4
- U1 pad 18: /Neopixel/GND -> GND
- U1 pad 19: /Key Matrix/Col 5 -> /Debounce Array/output 5
- U1 pad 21: E1-sw -> /RGB Encoder/Sw
- U1 pad 22: E1-A -> /RGB Encoder/enc B
- U1 pad 23: /Neopixel/GND -> GND
- U1 pad 24: E1-B -> /RGB Encoder/enc A
- U1 pad 25: E1-LED-B -> /RGB Encoder/LED-B
- U1 pad 26: E1-LED-G -> /RGB Encoder/LED-G
- U1 pad 27: E1-LED-R -> /RGB Encoder/LED-R
- U1 pad 28: /Neopixel/GND -> GND
- U1 pad 29: /Neopixel/DIN -> /Neopixel Logic Shifter/sigLOW
- U1 pad 3: /Neopixel/GND -> GND
- U1 pad 33: /Neopixel/GND -> GND
- U1 pad 36: unconnected-(U1-3V3-Pad36) -> /Neopixel Logic Shifter/3.3v
- U1 pad 7: /Key Matrix/Col 1 -> /Debounce Array/output 1
- U1 pad 8: /Neopixel/GND -> GND
- U1 pad 9: /Key Matrix/Col 2 -> /Debounce Array/output 2
Routing:
- net /Debounce Array/input 1: track 0.00 -> 156.7 mm, vias 0 -> 6
- net /Debounce Array/input 2: track 0.00 -> 143.2 mm, vias 0 -> 6
- net /Debounce Array/input 4: track 0.00 -> 127.3 mm, vias 0 -> 6
- net /Debounce Array/input 3: track 0.00 -> 113.8 mm, vias 0 -> 6
- net /Debounce Array/input 5: track 0.00 -> 112.5 mm, vias 0 -> 6
- net /Key Matrix/Col 1: track 86.4 -> 0.00 mm
- net /Key Matrix/Col 4: track 85.6 -> 0.00 mm
- net /Key Matrix/Col 3: track 85.6 -> 0.00 mm
- net /Key Matrix/Col 2: track 85.6 -> 0.00 mm
- net /Key Matrix/Col 5: track 64.2 -> 0.00 mm
- net Net-(LED30-DOUT): track 0.00 -> 54.4 mm
- net Net-(LED32-DOUT): track 0.00 -> 49.5 mm
- net /Debounce Array/output 3: track 0.00 -> 49.3 mm, vias 0 -> 1
- net /Debounce Array/output 2: track 0.00 -> 47.0 mm, vias 0 -> 1
- net Net-(LED27-DOUT): track 0.00 -> 46.7 mm
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Other:
- board size 3.8 x 3.4 mm -> 103 x 127.5 mm
