File: Roto-Pad-2.0/debounce.kicad_sch (KiCad schematic)
At the start: 10 parts

Commit message: layout completed, first draft of routing
Parts:
- C5, C6, C7, C8, C9: footprint (none) -> Keebio-Parts.pretty-master:C_0402
- R14, R15, R16, R17, R18: footprint (none) -> adafruit:R0805
Changed lines of the file:
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@@
 			)
 		)
-		(property "Footprint" ""
+		(property "Footprint" "adafruit:R0805"
 			(at 92.71 63.5 0)
 			(effects
@@
 			)
 		)
-		(property "Footprint" ""
+		(property "Footprint" "Keebio-Parts.pretty-master:C_0402"
 			(at 101.6 45.72 0)
 			(effects
@@
 			)
 		)
-		(property "Footprint" ""
+		(property "Footprint" "adafruit:R0805"
 			(at 92.71 139.7 0)
 			(effects
@@
 			)
 		)
-		(property "Footprint" ""
+		(property "Footprint" "adafruit:R0805"
 			(at 92.71 38.1 0)
 			(effects
@@
 			)
 		)
-		(property "Footprint" ""
+		(property "Footprint" "Keebio-Parts.pretty-master:C_0402"
 			(at 101.6 121.92 0)
 			(effects
@@
 			)
 		)
-		(property "Footprint" ""
+		(property "Footprint" "adafruit:R0805"
 			(at 92.71 114.3 0)
 			(effects
@@
 			)
 		)
-		(property "Footprint" ""
+		(property "Footprint" "Keebio-Parts.pretty-master:C_0402"
 			(at 101.6 96.52 0)
 			(effects
@@
 			)
 		)
-		(property "Footprint" ""
+		(property "Footprint" "Keebio-Parts.pretty-master:C_0402"
 			(at 101.6 147.32 0)
 			(effects
@@
 			)
 		)
-		(property "Footprint" ""
+		(property "Footprint" "adafruit:R0805"
 			(at 92.71 88.9 0)
 			(effects
@@
 			)
 		)
-		(property "Footprint" ""
+		(property "Footprint" "Keebio-Parts.pretty-master:C_0402"
 			(at 101.6 71.12 0)
 			(effects

Commit message: PCB passes DRC
Parts:
- R14, R15, R16, R17, R18: footprint adafruit:R0805 -> Custom:R0805
Changed lines of the file:
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@@
 			)
 		)
-		(property "Footprint" "adafruit:R0805"
+		(property "Footprint" "Custom:R0805"
 			(at 92.71 63.5 0)
 			(effects
@@
 			)
 		)
-		(property "Footprint" "adafruit:R0805"
+		(property "Footprint" "Custom:R0805"
 			(at 92.71 139.7 0)
 			(effects
@@
 			)
 		)
-		(property "Footprint" "adafruit:R0805"
+		(property "Footprint" "Custom:R0805"
 			(at 92.71 38.1 0)
 			(effects
@@
 			)
 		)
-		(property "Footprint" "adafruit:R0805"
+		(property "Footprint" "Custom:R0805"
 			(at 92.71 114.3 0)
 			(effects
@@
 			)
 		)
-		(property "Footprint" "adafruit:R0805"
+		(property "Footprint" "Custom:R0805"
 			(at 92.71 88.9 0)
 			(effects
