File: Roto-Pad-2.0/rgbencoder.kicad_sch (KiCad schematic)
At the start: 13 parts

Commit message: layout completed, first draft of routing
Parts:
- C10, C11: value C104 -> 10nf
- C12: footprint (none) -> Keebio-Parts.pretty-master:C_0402
- R19, R20, R21, R22: footprint PCM_Resistor_SMD_AKL:R_1206_3216Metric -> PCM_4ms_Resistor:R_0402
- R23: footprint (none) -> adafruit:R0805
- R24, R25, R26: footprint PCM_Resistor_SMD_AKL:R_1206_3216Metric -> adafruit:R1206
- R27: footprint (none) -> PCM_4ms_Resistor:R_0402
Changed lines of the file:
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@@
 			)
 		)
-		(property "Footprint" "PCM_Resistor_SMD_AKL:R_1206_3216Metric"
+		(property "Footprint" "adafruit:R1206"
 			(at 168.529 86.868 0)
 			(effects
@@
 			)
 		)
-		(property "Footprint" ""
+		(property "Footprint" "Keebio-Parts.pretty-master:C_0402"
 			(at 168.91 100.33 0)
 			(effects
@@
 			)
 		)
-		(property "Value" "C104"
+		(property "Value" "10nf"
 			(at 97.79 83.82 90)
 			(effects
@@
 			)
 		)
-		(property "Footprint" ""
+		(property "Footprint" "adafruit:R0805"
 			(at 162.56 95.25 0)
 			(effects
@@
 			)
 		)
-		(property "Footprint" "PCM_Resistor_SMD_AKL:R_1206_3216Metric"
+		(property "Footprint" "PCM_4ms_Resistor:R_0402"
 			(at 125.73 90.17 0)
 			(effects
@@
 			)
 		)
-		(property "Footprint" "PCM_Resistor_SMD_AKL:R_1206_3216Metric"
+		(property "Footprint" "PCM_4ms_Resistor:R_0402"
 			(at 111.76 74.93 0)
 			(effects
@@
 			)
 		)
-		(property "Footprint" "PCM_Resistor_SMD_AKL:R_1206_3216Metric"
+		(property "Footprint" "PCM_4ms_Resistor:R_0402"
 			(at 124.46 69.85 0)
 			(effects
@@
 			)
 		)
-		(property "Footprint" "PCM_Resistor_SMD_AKL:R_1206_3216Metric"
+		(property "Footprint" "adafruit:R1206"
 			(at 168.529 84.328 0)
 			(effects
@@
 			)
 		)
-		(property "Footprint" ""
+		(property "Footprint" "PCM_4ms_Resistor:R_0402"
 			(at 177.8 100.33 0)
 			(effects
@@
 			)
 		)
-		(property "Value" "C104"
+		(property "Value" "10nf"
 			(at 97.79 73.66 90)
 			(effects
@@
 			)
 		)
-		(property "Footprint" "PCM_Resistor_SMD_AKL:R_1206_3216Metric"
+		(property "Footprint" "PCM_4ms_Resistor:R_0402"
 			(at 111.76 85.09 0)
 			(effects
@@
 			)
 		)
-		(property "Footprint" "PCM_Resistor_SMD_AKL:R_1206_3216Metric"
+		(property "Footprint" "adafruit:R1206"
 			(at 168.529 89.408 0)
 			(effects

Commit message: PCB passes DRC
Parts:
- R23: footprint adafruit:R0805 -> Custom:R0805
Changed lines of the file:
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@@
 			)
 		)
-		(property "Footprint" "adafruit:R0805"
+		(property "Footprint" "Custom:R0805"
 			(at 162.56 95.25 0)
 			(effects
